File: MACH3_SIMPLE/hardware/01_power.kicad_sch (KiCad schematic)
At the start: 19 parts, among them J3 5V IN, J4 24V IN

Commit message: MACH3-SIMPLE A1: on-board 5 V, isolated VFD port, four A0 fixes
Power: the 5 V input terminal is gone. An LM2596S-5.0 buck makes +5V from
V24, and the whole supply sits in the top-right corner beside the 24 V
terminal, away from the MCU crystal and the port lines.

Spindle: new J5 (AVI ACM FWD REV DCM). Port 2 pins 7/8/9 go through a
74HC14 to a PC847; the VFD side runs from a B2412S isolated module with a
78L05 reference, a two-pole RC filter and an LM358 trimmed to 10.0 V. It
has its own SP_ACM pour, and the board is routed in two passes so no
board-side copper enters it; autoroute.py barrier checks that and fab.sh
refuses Gerbers without it.

Fixes to A0:
- Q1-Q6 had drain and source swapped; every relay was stuck on through
  the body diode. check_design.py now checks MOSFET orientation.
- The top-edge legends were reversed (+24 over 0V, +5 over MPG B, EMG over
  X home). Signals now follow the printed order, one word per screw.
- PC847 was on a SOIC-16 footprint no PC847 fits; now SMD DIP-16.
- The promised reverse diodes across the input opto LEDs were missing;
  added as D20-D25, with the input channels laid out per screw.

ERC 0, structural checks pass, DRC 0 errors / 0 unconnected / 0 parity,
barrier clean. Not built or powered.

Co-Authored-By: Claude Opus 5.5 <noreply@anthropic.com>
Claude-Session: https://claude.ai/code/session_01MByiLT2xCcbGPkgCYQy33q
Parts:
- removed D1: SS34 reverse, Diode_SMD:D_SMA, symbol Device:D_Schottky
- removed F1: 1A slow 1206, Fuse:Fuse_1206_3216Metric, symbol Device:Fuse
- removed J3: 5V IN, TerminalBlock_Phoenix:TerminalBlock_Phoenix_MKDS-1,5-2_1x02_P5.00mm_Horizontal, symbol Connector:Conn_01x02_Pin
- added C4: 47uF 50V, Capacitor_SMD:CP_Elec_6.3x7.7, symbol Device:C_Polarized
- added C5: 1uF 50V X7R, Capacitor_SMD:C_1206_3216Metric, symbol Device:C
- added D4: SS34 catch, Diode_SMD:D_SMA, symbol Device:D_Schottky
- added L1: 47uH 1.5A shielded, Inductor_SMD:L_12x12mm_H8mm, symbol Device:L
- added U4: LM2596S-5, Package_TO_SOT_SMD:TO-263-5_TabPin3, symbol Regulator_Switching:LM2596S-5
- C1: value 100uF 16V -> 220uF 16V low ESR
Connections:
- net +5V: now also L1.2, U4.4 (FB)
- net GND: now also J4.1 (Pin_1), C4.2, C5.2, D4.2 (A), U4.3 (GND), U4.5 (~{ON}/OFF); no longer J4.2 (Pin_2)
- net V24: now also C4.1, C5.1, U4.1 (VIN)
- net VIN24: now also J4.2 (Pin_2); no longer J4.1 (Pin_1)
- new net BUCK_SW: D4.1 (K), L1.1, U4.2 (OUT)
Other:
- note added: "5 V LOGIC SUPPLY - MADE ON BOARD FROM 24 V"
- note added: "Feeds the buffers, the optocoupler LEDs on the PC side, the MCU, the"
- note added: "POWER. 24 V from the cabinet; the 5 V rail is made on the board."
- note added: "RS232 transceiver and the handwheel. An LM2596S-5.0 buck off V24, so the"
- note added: "board takes one supply. About 0.4 W lost at 0.4 A, where a 7805 would burn 7.6 W."
- note removed: "5 V LOGIC SUPPLY"
- note removed: "Feeds the buffers, the optocoupler LEDs on the PC side, the MCU and"
- note removed: "POWER. Two supplies from the cabinet, exactly as the board in service."
- note removed: "the RS232 transceiver. F1 protects the board, not the supply."
- title: Power - 5 V and 24 V in -> Power - 24 V in, 5 V made on board

Commit message: MACH3-SIMPLE A1: design-review fixes and options
- Relay terminals labelled: RELAY A-F and NO/COM/NC per screw on the back
  silkscreen, RELAY A-F on the front (were on F.Fab only, not printed).
- R80-R85 4k7 -> 10k: 103 mW in a 100 mW 0603 on 24 V.
- Axis buffers fitted as 74AC245 (same pads) for opto-input drivers.
- J4 is 4-way: fused +24/0V for the sensors beside +24/0V in.
- C2 47 uF 50 V: 100 uF 50 V is not made in 6.3 x 7.7.
- Function labels (5V, 24V, SERIAL, A-F, 10V ADJ), test points GND/5V/24V
  and ACM/12V/AVI, dashed ISOLATED line round the VFD side, MCU heading
  moved beside the MCU.
- Buck switch node hand-drawn and locked: 14 mm top layer, no vias.
- F3 200 mA PTC on the handwheel +5V; 10 nF on MCU reset.
- Spare opto channel as VFD AUX output (port 2 pin 6); J5 is 6-way.
- autoroute.py keeps locked tracks through imports; route_one.py for a
  connection the router leaves open.

ERC 0, structural checks pass, DRC 0 errors / 0 unconnected / 0 parity,
barrier clean. Not built or powered.

Co-Authored-By: Claude Opus 5.5 <noreply@anthropic.com>
Claude-Session: https://claude.ai/code/session_01MByiLT2xCcbGPkgCYQy33q
Parts:
- removed J4: 24V IN, TerminalBlock_Phoenix:TerminalBlock_Phoenix_MKDS-1,5-2_1x02_P5.00mm_Horizontal, symbol Connector:Conn_01x02_Pin
- added J4: SENSORS / 24V IN, TerminalBlock_Phoenix:TerminalBlock_Phoenix_MKDS-1,5-4_1x04_P5.00mm_Horizontal, symbol Connector:Conn_01x04_Pin
- added TP1: GND, TestPoint:TestPoint_THTPad_D2.0mm_Drill1.0mm, symbol Connector:TestPoint
- added TP2: 5V, TestPoint:TestPoint_THTPad_D2.0mm_Drill1.0mm, symbol Connector:TestPoint
- added TP3: 24V, TestPoint:TestPoint_THTPad_D2.0mm_Drill1.0mm, symbol Connector:TestPoint
- C2: value 100uF 50V -> 47uF 50V
Connections:
- net +5V: now also TP2.1
- net GND: now also J4.1 (Pin_1), J4.3 (Pin_3), TP1.1
- net V24: now also J4.4 (Pin_4), TP3.1
- net VIN24: now also J4.2 (Pin_2)
Other:
- note added: "TEST POINTS"
