File: MACH3_SIMPLE/hardware/05_spindle.kicad_sch (KiCad schematic)
At the start: 27 parts, among them J5 VFD, U12 PC847, U13 B2412S-1WR3, U14 78L05, U15 LM358, U16 74HC14

Commit message: MACH3-SIMPLE A1: design-review fixes and options
- Relay terminals labelled: RELAY A-F and NO/COM/NC per screw on the back
  silkscreen, RELAY A-F on the front (were on F.Fab only, not printed).
- R80-R85 4k7 -> 10k: 103 mW in a 100 mW 0603 on 24 V.
- Axis buffers fitted as 74AC245 (same pads) for opto-input drivers.
- J4 is 4-way: fused +24/0V for the sensors beside +24/0V in.
- C2 47 uF 50 V: 100 uF 50 V is not made in 6.3 x 7.7.
- Function labels (5V, 24V, SERIAL, A-F, 10V ADJ), test points GND/5V/24V
  and ACM/12V/AVI, dashed ISOLATED line round the VFD side, MCU heading
  moved beside the MCU.
- Buck switch node hand-drawn and locked: 14 mm top layer, no vias.
- F3 200 mA PTC on the handwheel +5V; 10 nF on MCU reset.
- Spare opto channel as VFD AUX output (port 2 pin 6); J5 is 6-way.
- autoroute.py keeps locked tracks through imports; route_one.py for a
  connection the router leaves open.

ERC 0, structural checks pass, DRC 0 errors / 0 unconnected / 0 parity,
barrier clean. Not built or powered.

Co-Authored-By: Claude Opus 5.5 <noreply@anthropic.com>
Claude-Session: https://claude.ai/code/session_01MByiLT2xCcbGPkgCYQy33q
Parts:
- removed J5: VFD, TerminalBlock_Phoenix:TerminalBlock_Phoenix_MKDS-1,5-5_1x05_P5.00mm_Horizontal, symbol Connector:Conn_01x05_Pin
- added J5: VFD, TerminalBlock_Phoenix:TerminalBlock_Phoenix_MKDS-1,5-6_1x06_P5.00mm_Horizontal, symbol Connector:Conn_01x06_Pin
- added R102: 10k pull-down, Resistor_SMD:R_0603_1608Metric, symbol Device:R
- added R103: 330R, Resistor_SMD:R_0603_1608Metric, symbol Device:R
- added TP4: ACM, TestPoint:TestPoint_THTPad_D2.0mm_Drill1.0mm, symbol Connector:TestPoint
- added TP5: 12V, TestPoint:TestPoint_THTPad_D2.0mm_Drill1.0mm, symbol Connector:TestPoint
- added TP6: AVI, TestPoint:TestPoint_THTPad_D2.0mm_Drill1.0mm, symbol Connector:TestPoint
Connections:
- net +5V: now also R103.1
- net GND: now also R102.2; no longer U16.9
- net SP_12V: now also TP5.1
- net SP_ACM: now also J5.5 (Pin_5), TP4.1
- net SP_AVI: now also J5.6 (Pin_6), TP6.1
- net SP_DCM: now also U12.9, J5.1 (Pin_1)
- net SP_FWD: now also J5.4 (Pin_4)
- net SP_REV: now also J5.3 (Pin_3)
- net SP_AUX: now reaches U12.10
- net SP_AUX: now also J5.2 (Pin_2)
- net SP_AUX_A: now reaches U12.7
- net SP_AUX_A: now also R103.2
- net SP_AUX_K: now reaches U12.8
- net SP_AUX_K: now also U16.8
- new net SP_AUX_IN: R102.1, U16.9
- no-connect marks 7 -> 2
Other:
- note added: "AVI ACM FWD REV AUX DCM. Most VFDs ship with FWD/REV in NPN (sink) mode,"
- note added: "VFD-SIDE TEST POINTS - measure against ACM"
- note removed: "AVI ACM FWD REV DCM. Most VFDs ship with FWD/REV in NPN (sink) mode,"
