File: MACH3_SIMPLE/hardware/MACH3SIMPLE.kicad_pcb (KiCad board)
At the start: 2 copper layers, 150.5 x 137.9 mm, 133 parts, among them J1 LPT PORT 1, J10 X axis, J11 Y axis, J12 Z axis, J13 A axis, J14 B axis, J15 C axis, J2 LPT PORT 2, J20 EMG C A Z Y X, J3 5V IN, J30 MPG handwheel, J4 24V IN, J40 Relay A, J41 Relay B, J42 Relay C, J43 Relay D, J44 Relay E, J45 Relay F, J50 RS232 RX TX GND, J60 ICSP, K1 JQC-3FF-024-1Z, K2 JQC-3FF-024-1Z, K3 JQC-3FF-024-1Z, K4 JQC-3FF-024-1Z, K5 JQC-3FF-024-1Z, K6 JQC-3FF-024-1Z, Q1 2N7002, Q2 2N7002, Q3 2N7002, Q4 2N7002, Q5 2N7002, Q6 2N7002, U1 74HC245, U10 PC847, U11 PC847, U2 74HC245, U20 MAX3232, U21 ATmega328P-AU, U3 74HC4053, Y1 16MHz

Commit message: MACH3-SIMPLE A1: on-board 5 V, isolated VFD port, four A0 fixes
Power: the 5 V input terminal is gone. An LM2596S-5.0 buck makes +5V from
V24, and the whole supply sits in the top-right corner beside the 24 V
terminal, away from the MCU crystal and the port lines.

Spindle: new J5 (AVI ACM FWD REV DCM). Port 2 pins 7/8/9 go through a
74HC14 to a PC847; the VFD side runs from a B2412S isolated module with a
78L05 reference, a two-pole RC filter and an LM358 trimmed to 10.0 V. It
has its own SP_ACM pour, and the board is routed in two passes so no
board-side copper enters it; autoroute.py barrier checks that and fab.sh
refuses Gerbers without it.

Fixes to A0:
- Q1-Q6 had drain and source swapped; every relay was stuck on through
  the body diode. check_design.py now checks MOSFET orientation.
- The top-edge legends were reversed (+24 over 0V, +5 over MPG B, EMG over
  X home). Signals now follow the printed order, one word per screw.
- PC847 was on a SOIC-16 footprint no PC847 fits; now SMD DIP-16.
- The promised reverse diodes across the input opto LEDs were missing;
  added as D20-D25, with the input channels laid out per screw.

ERC 0, structural checks pass, DRC 0 errors / 0 unconnected / 0 parity,
barrier clean. Not built or powered.

Co-Authored-By: Claude Opus 5.5 <noreply@anthropic.com>
Claude-Session: https://claude.ai/code/session_01MByiLT2xCcbGPkgCYQy33q
Parts:
- removed D1: SS34 reverse, Diode_SMD:D_SMA
- removed F1: 1A slow 1206, Fuse:Fuse_1206_3216Metric
- removed J3: 5V IN, TerminalBlock_Phoenix:TerminalBlock_Phoenix_MKDS-1,5-2_1x02_P5.00mm_Horizontal
- added C4: 47uF 50V, Capacitor_SMD:CP_Elec_6.3x7.7, F.Cu at (113.0, 13.9)
- added C5: 1uF 50V X7R, Capacitor_SMD:C_1206_3216Metric, F.Cu at (106.6, 16.0)
- added C60: 100nF, Capacitor_SMD:C_0603_1608Metric, F.Cu at (22.0, 83.8)
- added C61: 1uF 50V X7R, Capacitor_SMD:C_1206_3216Metric, F.Cu at (43.0, 38.5)
- added C62: 10uF 25V X7R, Capacitor_SMD:C_1206_3216Metric, F.Cu at (36.8, 23.5)
- added C63: 1uF, Capacitor_SMD:C_0603_1608Metric, F.Cu at (28.0, 27.4)
- added C64: 470nF, Capacitor_SMD:C_0603_1608Metric, F.Cu at (27.0, 30.0)
- added C65: 470nF, Capacitor_SMD:C_0603_1608Metric, F.Cu at (35.0, 30.0)
- added C66: 100nF, Capacitor_SMD:C_0603_1608Metric, F.Cu at (21.5, 24.5)
- added C67: 10nF, Capacitor_SMD:C_0603_1608Metric, F.Cu at (22.8, 15.9)
- added D20: 1N4148 LED reverse, Diode_SMD:D_SOD-123, F.Cu at (53.5, 19.6)
- added D21: 1N4148 LED reverse, Diode_SMD:D_SOD-123, F.Cu at (58.6, 19.6)
- added D22: 1N4148 LED reverse, Diode_SMD:D_SOD-123, F.Cu at (63.7, 19.6)
- added D23: 1N4148 LED reverse, Diode_SMD:D_SOD-123, F.Cu at (68.7, 19.6)
- added D24: 1N4148 LED reverse, Diode_SMD:D_SOD-123, F.Cu at (75.2, 19.6)
- added D25: 1N4148 LED reverse, Diode_SMD:D_SOD-123, F.Cu at (80.2, 19.6)
- added D4: SS34 catch, Diode_SMD:D_SMA, F.Cu at (101.5, 23.9)
- added J5: VFD, TerminalBlock_Phoenix:TerminalBlock_Phoenix_MKDS-1,5-5_1x05_P5.00mm_Horizontal, F.Cu at (37.0, 3.80)
- added L1: 47uH 1.5A shielded, Inductor_SMD:L_12x12mm_H8mm, F.Cu at (99.0, 37.0)
- added R100: 8k2, Resistor_SMD:R_0603_1608Metric, F.Cu at (26.0, 20.0)
- added R101: 100R, Resistor_SMD:R_0603_1608Metric, F.Cu at (18.5, 15.9)
- added R90: 10k pull-down, Resistor_SMD:R_0603_1608Metric, F.Cu at (18.0, 96.8)
- added R91: 10k pull-down, Resistor_SMD:R_0603_1608Metric, F.Cu at (22.0, 96.8)
- added R92: 10k pull-down, Resistor_SMD:R_0603_1608Metric, F.Cu at (26.0, 96.8)
- added R93: 330R, Resistor_SMD:R_0603_1608Metric, F.Cu at (18.6, 47.3)
- added R94: 330R, Resistor_SMD:R_0603_1608Metric, F.Cu at (23.7, 47.3)
- added R95: 330R, Resistor_SMD:R_0603_1608Metric, F.Cu at (28.8, 47.3)
- added R96: 2k2, Resistor_SMD:R_0603_1608Metric, F.Cu at (19.0, 30.0)
- added R97: 100k, Resistor_SMD:R_0603_1608Metric, F.Cu at (23.0, 30.0)
- added R98: 100k, Resistor_SMD:R_0603_1608Metric, F.Cu at (31.0, 30.0)
- added R99: 10k, Resistor_SMD:R_0603_1608Metric, F.Cu at (26.0, 24.5)
- added RV1: 5k 10.0V trim, Potentiometer_THT:Potentiometer_Bourns_3296W_Vertical, F.Cu at (36.0, 18.0)
- added U12: PC847, Package_DIP:SMDIP-16_W9.53mm, F.Cu at (27.5, 38.5)
- added U13: B2412S-1WR3, Converter_DCDC:Converter_DCDC_Murata_CRE1xxxxxxSC_THT, F.Cu at (43.5, 33.5)
- added U14: 78L05, Package_TO_SOT_SMD:SOT-89-3, F.Cu at (32.0, 24.0)
- added U15: LM358, Package_SO:SOIC-8_3.9x4.9mm_P1.27mm, F.Cu at (21.0, 20.0)
- added U16: 74HC14, Package_SO:SOIC-14_3.9x8.7mm_P1.27mm, F.Cu at (22.0, 90.0)
- added U4: LM2596S-5, Package_TO_SOT_SMD:TO-263-5_TabPin3, F.Cu at (113.5, 24.1)
- C1: value 100uF 16V -> 220uF 16V low ESR
- U10, U11: footprint Package_SO:SOIC-16_3.9x9.9mm_P1.27mm -> Package_DIP:SMDIP-16_W9.53mm
- moved R15 46.3 mm to (80.2, 15.9)
- moved R35 38.9 mm to (80.2, 36.6), turned to 90 degrees
- moved R43 37.7 mm to (51.7, 55.1)
- moved R42 33.4 mm to (45.9, 55.1)
- moved F2 32.8 mm to (118.0, 6.00)
- moved R41 29.4 mm to (40.1, 55.1)
- moved C13 28.5 mm to (71.3, 36.6), turned to 90 degrees
- moved C12 28.4 mm to (66.2, 36.6), turned to 90 degrees
- moved C11 28.3 mm to (61.1, 36.6), turned to 90 degrees
- moved C10 28.2 mm to (56.0, 36.6), turned to 90 degrees
- moved R2 27.4 mm to (133.0, 33.8)
- moved R40 25.6 mm to (34.3, 55.1)
- moved C14 22.1 mm to (77.7, 36.6), turned to 90 degrees
- moved C15 21.3 mm to (82.8, 36.6), turned to 90 degrees
- moved D3 21.1 mm to (126.0, 31.0)
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Connections:
- J2 pad 7: unconnected-(J2-Pad7) -> SP_PWM_IN
- J2 pad 8: unconnected-(J2-Pad8) -> SP_FWD_IN
- J2 pad 9: unconnected-(J2-Pad9) -> SP_REV_IN
- J20 pad 1: ESTOP_F -> X_HOME_F
- J20 pad 2: C_HOME_F -> Y_HOME_F
- J20 pad 3: A_HOME_F -> Z_HOME_F
- J20 pad 4: Z_HOME_F -> A_HOME_F
- J20 pad 5: Y_HOME_F -> C_HOME_F
- J20 pad 6: X_HOME_F -> ESTOP_F
- J30 pad 1: +5V -> MPG_B_RAW
- J30 pad 2: GND -> MPG_A_RAW
- J30 pad 3: MPG_A_RAW -> GND
- J30 pad 4: MPG_B_RAW -> +5V
- J4 pad 1: VIN24 -> GND
- J4 pad 2: GND -> VIN24
- Q1 pad 2: RELC_A -> GND
- Q1 pad 3: GND -> RELC_A
- Q2 pad 2: RELC_B -> GND
- Q2 pad 3: GND -> RELC_B
- Q3 pad 2: RELC_C -> GND
- Q3 pad 3: GND -> RELC_C
- Q4 pad 2: RELC_D -> GND
- Q4 pad 3: GND -> RELC_D
- Q5 pad 2: RELC_E -> GND
- Q5 pad 3: GND -> RELC_E
- Q6 pad 2: RELC_F -> GND
- Q6 pad 3: GND -> RELC_F
- U10 pad 1: ESTOP_LED -> Z_HOME_LED
- U10 pad 10: Z_HOME_PC -> ESTOP_PC
- U10 pad 12: A_HOME_PC -> C_HOME_PC
- U10 pad 14: C_HOME_PC -> A_HOME_PC
- U10 pad 16: ESTOP_PC -> Z_HOME_PC
- U10 pad 3: C_HOME_LED -> A_HOME_LED
- U10 pad 5: A_HOME_LED -> C_HOME_LED
- U10 pad 7: Z_HOME_LED -> ESTOP_LED
- U11 pad 1: Y_HOME_LED -> unconnected-(U11-Pad1)
- U11 pad 10: unconnected-(U11-Pad10) -> Y_HOME_PC
- U11 pad 11: unconnected-(U11-Pad11) -> GND
- U11 pad 12: unconnected-(U11-Pad12) -> X_HOME_PC
- U11 pad 13: GND -> unconnected-(U11-Pad13)
- U11 pad 14: X_HOME_PC -> unconnected-(U11-Pad14)
- U11 pad 15: GND -> unconnected-(U11-Pad15)
- U11 pad 16: Y_HOME_PC -> unconnected-(U11-Pad16)
- U11 pad 2: GND -> unconnected-(U11-Pad2)
- U11 pad 3: X_HOME_LED -> unconnected-(U11-Pad3)
- U11 pad 4: GND -> unconnected-(U11-Pad4)
- U11 pad 5: unconnected-(U11-Pad5) -> X_HOME_LED
- U11 pad 6: unconnected-(U11-Pad6) -> GND
- U11 pad 7: unconnected-(U11-Pad7) -> Y_HOME_LED
- U11 pad 8: unconnected-(U11-Pad8) -> GND
- U11 pad 9: unconnected-(U11-Pad9) -> GND
Routing:
- net GND: track 910.4 -> 1029.8 mm, vias 132 -> 137
- net V24: track 364.8 -> 467.4 mm, vias 10 -> 12
- net SP_ACM: track 0.00 -> 97.0 mm, vias 0 -> 1
- net MPG_B_RAW: track 49.2 -> 118.4 mm, vias 1 -> 3
- net SP_REV_K: track 0.00 -> 61.5 mm, vias 0 -> 2
- net +5V: track 399.7 -> 455.0 mm, vias 7 -> 15
- net ESTOP_F: track 65.3 -> 12.8 mm, vias 2 -> 0
- net SP_FWD_K: track 0.00 -> 50.7 mm, vias 0 -> 2
- net MPG_A_RAW: track 66.2 -> 116.8 mm, vias 1 -> 3
- net SP_FWD: track 0.00 -> 45.5 mm, vias 0 -> 1
- net SP_PWM_K: track 0.00 -> 45.2 mm, vias 0 -> 2
- net SP_12V: track 0.00 -> 42.2 mm
- net VIN5: track 42.0 -> 0.00 mm, vias 1 -> 0
- net X_HOME_LED: track 49.3 -> 10.3 mm
- net SP_DCM: track 0.00 -> 38.5 mm, vias 0 -> 1
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- added copper zone on B.Cu, net SP_ACM
- added copper zone on F.Cu, net SP_ACM
Other:
- board text added: "+24"
- board text added: "+5"
- board text added: "0V"
- board text added: "5V BUCK"
- board text added: "A"
- board text added: "ACM"
- board text added: "AVI"
- board text added: "B"
- board text added: "C"
- board text added: "DCM"
- board text added: "EMG"
- board text added: "FWD"
- board text added: "MACH3-SIMPLE A1"
- board text added: "NOT ISOLATED - EXCEPT THE VFD PORT"
- board text added: "REV"
- board text added: "VFD - ISOLATED"
- board text added: "X"
- board text added: "Y"
- board text added: "Z"
- board text removed: "+24 0V"
- board text removed: "+5 0V"
- board text removed: "+5 0V A B"
- board text removed: "5V IN"
- board text removed: "EMG C A Z Y X"
- board text removed: "INPUTS"
- board text removed: "MACH3-SIMPLE NOT ISOLATED"

Commit message: MACH3-SIMPLE A1: design-review fixes and options
- Relay terminals labelled: RELAY A-F and NO/COM/NC per screw on the back
  silkscreen, RELAY A-F on the front (were on F.Fab only, not printed).
- R80-R85 4k7 -> 10k: 103 mW in a 100 mW 0603 on 24 V.
- Axis buffers fitted as 74AC245 (same pads) for opto-input drivers.
- J4 is 4-way: fused +24/0V for the sensors beside +24/0V in.
- C2 47 uF 50 V: 100 uF 50 V is not made in 6.3 x 7.7.
- Function labels (5V, 24V, SERIAL, A-F, 10V ADJ), test points GND/5V/24V
  and ACM/12V/AVI, dashed ISOLATED line round the VFD side, MCU heading
  moved beside the MCU.
- Buck switch node hand-drawn and locked: 14 mm top layer, no vias.
- F3 200 mA PTC on the handwheel +5V; 10 nF on MCU reset.
- Spare opto channel as VFD AUX output (port 2 pin 6); J5 is 6-way.
- autoroute.py keeps locked tracks through imports; route_one.py for a
  connection the router leaves open.

ERC 0, structural checks pass, DRC 0 errors / 0 unconnected / 0 parity,
barrier clean. Not built or powered.

Co-Authored-By: Claude Opus 5.5 <noreply@anthropic.com>
Claude-Session: https://claude.ai/code/session_01MByiLT2xCcbGPkgCYQy33q
Parts:
- added C35: 10nF, Capacitor_SMD:C_0603_1608Metric, F.Cu at (61.5, 61.0)
- added F3: 200mA hold PTC 1206, Fuse:Fuse_1206_3216Metric, F.Cu at (87.0, 14.5)
- added R102: 10k pull-down, Resistor_SMD:R_0603_1608Metric, F.Cu at (30.0, 96.8)
- added R103: 330R, Resistor_SMD:R_0603_1608Metric, F.Cu at (33.9, 47.3)
- added TP1: GND, TestPoint:TestPoint_THTPad_D2.0mm_Drill1.0mm, F.Cu at (118.5, 37.5)
- added TP2: 5V, TestPoint:TestPoint_THTPad_D2.0mm_Drill1.0mm, F.Cu at (121.5, 37.5)
- added TP3: 24V, TestPoint:TestPoint_THTPad_D2.0mm_Drill1.0mm, F.Cu at (122.0, 24.5)
- added TP4: ACM, TestPoint:TestPoint_THTPad_D2.0mm_Drill1.0mm, F.Cu at (40.5, 15.0)
- added TP5: 12V, TestPoint:TestPoint_THTPad_D2.0mm_Drill1.0mm, F.Cu at (43.5, 15.0)
- added TP6: AVI, TestPoint:TestPoint_THTPad_D2.0mm_Drill1.0mm, F.Cu at (40.5, 19.5)
- C2: value 100uF 50V -> 47uF 50V
- J4: value 24V IN -> SENSORS / 24V IN; footprint TerminalBlock_Phoenix:TerminalBlock_Phoenix_MKDS-1,5-2_1x02_P5.00mm_Horizontal -> TerminalBlock_Phoenix:TerminalBlock_Phoenix_MKDS-1,5-4_1x04_P5.00mm_Horizontal
- J5: footprint TerminalBlock_Phoenix:TerminalBlock_Phoenix_MKDS-1,5-5_1x05_P5.00mm_Horizontal -> TerminalBlock_Phoenix:TerminalBlock_Phoenix_MKDS-1,5-6_1x06_P5.00mm_Horizontal
- R80, R81, R82, R83, R84, R85: value 4k7 -> 10k
- U1, U2: value 74HC245 -> 74AC245
- moved R50 28.9 mm to (95.3, 61.0)
- moved F2 11.7 mm to (122.0, 17.0), turned to 90 degrees
- moved D30 4.96 mm to (66.4, 61.0)
- moved R51 4.54 mm to (104.4, 61.0)
- moved J5 4.00 mm to (41.0, 3.80)
- moved C4 3.27 mm to (110.0, 15.2)
- moved D4 3.08 mm to (98.5, 24.6), turned to 90 degrees
- moved U4 3.08 mm to (110.5, 24.8)
- moved C5 2.63 mm to (104.0, 16.4)
- moved L1 0.40 mm to (99.0, 37.4)
- moved J4 0.05 mm to (131.6, 3.80)
Connections:
- J2 pad 6: unconnected-(J2-Pad6) -> SP_AUX_IN
- J30 pad 4: +5V -> MPG_5V
- J5 pad 2: SP_REV -> SP_AUX
- J5 pad 3: SP_FWD -> SP_REV
- J5 pad 4: SP_ACM -> SP_FWD
- J5 pad 5: SP_AVI -> SP_ACM
- U12 pad 10: unconnected-(U12-Pad10) -> SP_AUX
- U12 pad 7: unconnected-(U12-Pad7) -> SP_AUX_A
- U12 pad 8: unconnected-(U12-Pad8) -> SP_AUX_K
- U12 pad 9: unconnected-(U12-Pad9) -> SP_DCM
- U16 pad 8: unconnected-(U16-Pad8) -> SP_AUX_K
- U16 pad 9: GND -> SP_AUX_IN
Routing:
- net SP_AUX_K: track 0.00 -> 58.2 mm, vias 0 -> 2
- net MCU_RESET: track 41.8 -> 84.2 mm, vias 2 -> 4
- net +5V: track 455.0 -> 492.7 mm, vias 15 -> 14
- net SP_AUX: track 0.00 -> 30.8 mm, vias 0 -> 1
- net ESTOP_PC: track 133.2 -> 104.4 mm
- net SP_AUX_IN: track 0.00 -> 28.7 mm
- net SP_AVI: track 15.8 -> 42.8 mm
- net MCU_TX: track 115.0 -> 135.8 mm
- net MPG_A_RAW: track 116.8 -> 99.7 mm, vias 3 -> 1
- net B_PUL_IN: track 144.6 -> 161.2 mm
- net Y_PUL_IN: track 119.1 -> 135.6 mm
- net MPG_B_THC: track 69.8 -> 53.6 mm, vias 1 -> 2
- net Y_DIR_IN: track 138.9 -> 123.8 mm, vias 2 -> 0
- net C_HOME_PC: track 66.7 -> 81.2 mm, vias 0 -> 2
- net Net-(Q6-G): track 70.0 -> 84.0 mm
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Other:
- board text added: "10V ADJ"
- board text added: "12V"
- board text added: "24V"
- board text added: "5V"
- board text added: "AUX"
- board text added: "COM"
- board text added: "D"
- board text added: "E"
- board text added: "F"
- board text added: "GND"
- board text added: "ISOLATED"
- board text added: "NC"
- board text added: "NO"
- board text added: "SENSORS 24V IN"
- board text added: "SERIAL"
- board text removed: "24V IN"
