File: MACH3_SIMPLE_ETH/hardware/01_power.kicad_sch (KiCad schematic)
At the start: 33 parts, among them J101 SENSORS / 24V IN, U101 LM2596S-5, U102 AP7361C-33E

Commit message: MACH3-SIMPLE-ETH: bare mounting holes, VBUS/CHASSIS parts moved to their connectors
After pass 2, 16 connections were left. Three were CHASSIS between the
corner mounting holes, which needed a track round the whole board edge:
the holes are bare now, as on A1, and the shield bond is at the magjack and
USB. Three were VBUS, because the auto-placer had put D104 in the middle
of the board. tools/autoroute.py fixup brings the routed board up to the
regenerated schematic (paths, holes), moves D104/C108/R104 next to the pads
they serve, clears the tracks they now sit on, and adds In2 ground pours so
stitching vias can land in ground on every layer. Parity 0.

Co-Authored-By: Claude Opus 5.5 <noreply@anthropic.com>
Claude-Session: https://claude.ai/code/session_01MByiLT2xCcbGPkgCYQy33q
Parts:
- removed H101, H102, H103, H104: M3, MountingHole:MountingHole_3.2mm_M3_Pad_Via, symbol Mechanical:MountingHole_Pad
- added H101, H102, H103, H104: M3, MountingHole:MountingHole_3.2mm_M3, symbol Mechanical:MountingHole
Other:
- note added: "Magjack and USB shields are CHASSIS; the mounting holes are bare."
- note removed: "Magjack shield, USB shield and mounting holes are CHASSIS."
