File: MACH3_SIMPLE_ETH/hardware/MACH3SIMPLEETH.kicad_pcb (KiCad board)
At the start: 4 copper layers, 210 x 155 mm, 337 parts, among them J101 SENSORS / 24V IN, J201 USB-C, J202 SWD, J203 microSD, J301 HR911105A, J401 X axis, J402 Y axis, J403 Z axis, J404 A axis, J405 B axis, J406 C axis, J407 U axis, J408 V axis, J409 ENABLE, J501 LIMITS X Y Z A B C U V, J502 EST HLD RUN PRB, J503 THC AOK UP DN, J601 EXPANSION, J611 Relay A, J612 Relay B, J613 Relay C, J614 Relay D, J615 Relay E, J616 Relay F, J701 VFD, J801 RS485 A B GND, J802 HW ICSP, J803 MPG PENDANT, K601 JQC-3FF-024-1Z, K602 JQC-3FF-024-1Z, K603 JQC-3FF-024-1Z, K604 JQC-3FF-024-1Z, K605 JQC-3FF-024-1Z, K606 JQC-3FF-024-1Z, Q601 AO3400A, Q602 AO3400A, Q603 AO3400A, Q604 AO3400A, Q605 AO3400A, Q606 AO3400A, SW201 RESET, SW202 BOOTSEL, U101 LM2596S-5, U102 AP7361C-33E, U201 RP2350B, U202 W25Q128JVS, U203 USBLC6-2SC6, U301 W5500, U401 74ACT245, U402 74ACT245, U403 74ACT245, U501 PC847, U502 PC847, U503 PC847, U504 PC847, U601 MCP23017-E/SO, U701 74HCT14, U702 PC847, U703 B2412S-1WR3, U704 78L05, U705 LM358, U801 MAX3485ESA, U802 ATmega328P-AU, Y201 12MHz ABM8-272-T3, Y301 25MHz 18pF, Y801 8MHz

Commit message: MACH3-SIMPLE-ETH: board snapshot during the rip-up repair run (intermediate)
Co-Authored-By: Claude Opus 5.5 <noreply@anthropic.com>
Claude-Session: https://claude.ai/code/session_01MByiLT2xCcbGPkgCYQy33q
Routing:
- net GND: track 723.2 -> 732.8 mm
- net Y_LIM: track 104.8 -> 100.0 mm
- net XIN: track 11.0 -> 6.91 mm
- net XOUT: track 4.02 -> 0.72 mm
- net VREG_LX: track 4.45 -> 1.38 mm
- net SP_FWD_IN: track 40.3 -> 37.4 mm
- net ETH_TXP: track 8.13 -> 5.40 mm
- net ETH_RXN: track 13.2 -> 11.2 mm
- net VBUS: track 12.1 -> 13.3 mm
- net VREG_AVDD: track 22.6 -> 21.5 mm
- net +3V3A: track 99.8 -> 98.7 mm
- net +3V3: track 704.9 -> 703.9 mm
- net X_LIM: track 112.0 -> 111.4 mm
Changed lines of the file:
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@@
 	)
 	(segment
-		(start 64.2487 80.2231)
-		(end 64.6 80.5744)
-		(width 0.2002)
-		(layer "F.Cu")
-		(net "+3V3")
-	)
-	(segment
 		(start 97.3412 57.2338)
 		(end 98.325 56.25)
@@
 	)
 	(segment
-		(start 64.6 80.5744)
-		(end 64.6 81.05)
-		(width 0.2002)
-		(layer "F.Cu")
-		(net "+3V3")
-	)
-	(segment
 		(start 41.898 78.857)
 		(end 41.23 79.525)
@@
 	)
 	(segment
-		(start 65.8004 81.0496)
-		(end 65.8 81.05)
-		(width 0.2002)
-		(layer "F.Cu")
-		(net "VREG_AVDD")
-	)
-	(segment
-		(start 65.8004 80.3759)
-		(end 65.8004 81.0496)
-		(width 0.2002)
-		(layer "F.Cu")
-		(net "VREG_AVDD")
-	)
-	(segment
-		(start 65.8004 80.3759)
-		(end 65.8004 79.9234)
-		(width 0.3)
-		(layer "F.Cu")
-		(net "VREG_AVDD")
-	)
-	(segment
 		(start 61.3645 98)
 		(end 61.5452 97.8193)
@@
 	)
 	(segment
+		(start 34.5 63.2)
+		(end 38.6 63.2)
+		(width 0.2)
+		(layer "F.Cu")
+		(net "GND")
+	)
+	(segment
 		(start 36.25 107.225)
 		(end 40.2602 111.235)
@@
 	)
 	(segment
+		(start 38.6 63.2)
+		(end 38.8 63)
+		(width 0.2)
+		(layer "F.Cu")
+		(net "GND")
+	)
+	(segment
 		(start 95.103 22.528)
 		(end 93.81 21.235)
@@
 	)
 	(segment
+		(start 62.9 77.3)
+		(end 62.9 76.5)
+		(width 0.2)
+		(layer "F.Cu")
+		(net "GND")
+	)
+	(segment
 		(start 20.275 121)
 		(end 20.275 120.95)
@@
 	)
 	(segment
+		(start 65.4 80.3)
+		(end 64.8 79.7)
+		(width 0.2)
+		(layer "F.Cu")
+		(net "GND")
+	)
+	(segment
 		(start 92.5573 29.5123)
 		(end 90.4219 29.5123)
@@
 	)
 	(segment
+		(start 64.8 79.7)
+		(end 64.8 79.2)
+		(width 0.2)
+		(layer "F.Cu")
+		(net "GND")
+	)
+	(segment
 		(start 43.4 107.6)
 		(end 44.0517 107.6)
@@
 	)
 	(segment
+		(start 65.4 80.7)
+		(end 65.4 80.3)
+		(width 0.2)
+		(layer "F.Cu")
+		(net "GND")
+	)
+	(segment
 		(start 91.3031 32.8989)
 		(end 90.837 32.8989)
@@
 		(net "GND")
 	)
+	(segment
+		(start 64.8 79.2)
+		(end 62.9 77.3)
+		(width 0.2)
+		(layer "F.Cu")
+		(net "GND")
+	)
 	(via
 		(at 57.3222 79.5152)
@@
 	)
 	(via
-		(at 69.6 90.9)
+		(at 38.8 63)
 		(size 0.6)
 		(drill 0.3)
@@
 	)
 	(via
-		(at 31.2 61.1)
+		(at 62.9 76.5)
 		(size 0.6)
 		(drill 0.3)
@@
 	)
 	(via
-		(at 69.6104 90.6476)
+		(at 69.6 90.9)
 		(size 0.6)
 		(drill 0.3)
@@
 	)
 	(via
-		(at 36.3117 67.5367)
+		(at 31.2 61.1)
 		(size 0.6)
 		(drill 0.3)
@@
 	)
 	(via
-		(at 31.2 61.1)
+		(at 36.3117 67.5367)
 		(size 0.6)
 		(drill 0.3)
@@
 	)
 	(segment
-		(start 60.6 90.95)
-		(end 60.6 91.5676)
-		(width 0.2)
-		(layer "F.Cu")
-		(net "X_LIM")
-	)
-	(segment
 		(start 51.2863 93.7655)
 		(end 50.6461 93.1253)
@@
 	)
 	(segment
-		(start 33.8375 62.75)
-		(end 31.1014 62.75)
-		(width 0.2)
-		(layer "F.Cu")
-		(net "ETH_TXP")
-	)
-	(segment
 		(start 29.384 62.2589)
 		(end 28.947 61.8219)
@@
 	)
 	(segment
-		(start 61 90.95)
-		(end 61 90.5052)
-		(width 0.2)
-		(layer "F.Cu")
-		(net "Y_LIM")
-	)
-	(segment
 		(start 62.19 21.235)
 		(end 60.8839 19.9289)
@@
 	)
 	(segment
-		(start 61.2507 90.2545)
-		(end 61.5015 90.2545)
-		(width 0.2)
-		(layer "F.Cu")
-		(net "Y_LIM")
-	)
-	(segment
 		(start 58.501 20.2787)
 		(end 58.501 22.2547)
@@
 	)
 	(segment
-		(start 61.5015 90.2545)
-		(end 64.1598 87.5962)
-		(width 0.2)
-		(layer "F.Cu")
-		(net "Y_LIM")
-	)
-	(segment
 		(start 62.2038 58.7298)
 		(end 62.425 58.7298)
@@
 		(net "Y_LIM")
 	)
-	(segment
-		(start 61 90.5052)
-		(end 61.2507 90.2545)
-		(width 0.2)
-		(layer "F.Cu")
-		(net "Y_LIM")
-	)
 	(via
 		(at 61.7623 23.2506)
@@
 	)
 	(segment
-		(start 61.8 95.0093)
-		(end 61.8 90.95)
-		(width 0.2)
-		(layer "F.Cu")
-		(net "XIN")
-	)
-	(segment
 		(start 66.3118 96.5118)
 		(end 66.65 96.85)
@@
 	)
 	(segment
-		(start 62.2 90.95)
-		(end 62.1668 90.9832)
-		(width 0.2)
-		(layer "F.Cu")
-		(net "XOUT")
-	)
-	(segment
-		(start 62.1668 90.9832)
-		(end 62.1668 94.2418)
-		(width 0.2)
-		(layer "F.Cu")
-		(net "XOUT")
-	)
-	(segment
 		(start 62.1668 94.2418)
 		(end 62.675 94.75)
@@
 	)
 	(segment
-		(start 65.8976 83.6405)
-		(end 65.8976 81.8446)
-		(width 0.2)
-		(layer "F.Cu")
-		(net "SP_FWD_IN")
-	)
-	(segment
 		(start 57.525 50.73)
 		(end 59.1123 50.73)
@@
 	)
 	(segment
-		(start 65.8976 81.8446)
-		(end 66.6402 81.102)
-		(width 0.2)
-		(layer "F.Cu")
-		(net "SP_FWD_IN")
-	)
-	(segment
 		(start 66.6402 81.102)
 		(end 66.6402 77.4735)
@@
 	)
 	(segment
-		(start 65 80.3755)
-		(end 65 81.05)
-		(width 0.2002)
-		(layer "F.Cu")
-		(net "VREG_LX")
-	)
-	(segment
 		(start 65 77.975)
 		(end 64.025 77)
@@
 	)
 	(segment
-		(start 65 80.3755)
-		(end 65 77.975)
-		(width 0.3)
-		(layer "F.Cu")
-		(net "VREG_LX")
-	)
-	(segment
 		(start 63.6922 79.9467)
 		(end 63.6922 79.7402)
@@
 	)
 	(segment
-		(start 32.7574 63.7995)
-		(end 33.788 63.7995)
-		(width 0.225)
-		(layer "F.Cu")
-		(net "+3V3A")
-	)
-	(segment
 		(start 34.6808 67.25)
 		(end 35.1434 67.7126)
@@
 	)
 	(segment
-		(start 33.788 63.7995)
-		(end 33.8375 63.75)
-		(width 0.225)
-		(layer "F.Cu")
-		(net "+3V3A")
-	)
-	(segment
 		(start 33.8375 67.25)
 		(end 34.6808 67.25)
@@
 	)
 	(segment
-		(start 34.827 63.9855)
-		(end 34.827 62.0262)
-		(width 0.2)
-		(layer "F.Cu")
-		(net "ETH_RXN")
-	)
-	(segment
 		(start 30.1647 64.4694)
 		(end 28.7056 64.4694)
@@
 	)
 	(segment
-		(start 6.4 76.7)
-		(end 6.4 78.5)
+		(start 6.4 78.7)
+		(end 6.4 76.7)
 		(width 0.2)
 		(layer "F.Cu")
@@
 	)
 	(segment
-		(start 7.8 79.2)
-		(end 7.3 79.7)
+		(start 8 79.2)
+		(end 6.9 79.2)
 		(width 0.2)
 		(layer "F.Cu")
@@
 	)
 	(segment
-		(start 6.4 78.5)
-		(end 7 79.1)
+		(start 7.8 79.2)
+		(end 7.3 79.7)
 		(width 0.2)
 		(layer "F.Cu")
@@
 		(width 0.2)
 		(layer "F.Cu")
+		(net "VBUS")
+	)
+	(segment
+		(start 6.9 79.2)
+		(end 6.4 78.7)
+		(width 0.2)
+		(layer "F.Cu")
